File: ltc2208-adc.kicad_sch (KiCad schematic)
At the start: 75 parts, among them J2 Conn_02x20_Odd_Even, U1 SN65EPT22, U2 LTC2208, U3 LT1117-3.3, U4 LT1117-ADJ, X1 122.88 MHz

Commit message: Clarified VCCIO issue
Parts:
- R31, R32: value R -> 121
Connections:
- net at TR1.5: now also R5.1
Other:
- note added: "configured for 2.5V"
Changed lines of the file:
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@@
 		)
 	)
+	(text "configured for 2.5V"
+		(exclude_from_sim no)
+		(at 271.78 66.802 0)
+		(effects
+			(font
+				(size 1.27 1.27)
+			)
+		)
+	)
 	(label "D13_P"
 		(at 204.47 54.61 0)
@@
 			)
 		)
-		(property "Value" "R"
+		(property "Value" "121"
 			(at 268.478 81.2221 0)
 			(effects
@@
 			)
 		)
-		(property "Value" "R"
+		(property "Value" "121"
 			(at 268.478 90.1121 0)
 			(effects
